Commit message: Fixed kinematic transformation for robot description. Added .urdf file generated from xacro, and also added the urdf graphtree. Fixed the possitions and directions of the robot wheels.

File: urdf/jimmbot.xacro (robot description, xacro)
@@ -98,16 +98,16 @@
     </link>
     <joint name="chassis_to_boggie_${postfix}" type="revolute">
-        <axis xyz="1 0 0"/>
+        <axis xyz="${reflect*-1} 0 0"/>
         <limit effort="1000.0" lower="-0.523599" upper="0.523599" velocity="50"/>
-        <origin rpy="0 0 ${reflect*-1.57}" xyz="0 ${reflect*0.3} 0"/>
+        <origin rpy="0 0 ${reflect*1.57}" xyz="-1.45758E-03 ${reflect*-201.552E-03} -19.8088E-03"/>
         <parent link="chassis"/>
         <child link="boggie_${postfix}"/>
     </joint>
 </xacro:macro>
-<xacro:boggie postfix="right" reflect="-1" />
-<xacro:boggie postfix="left" reflect="1" />
+<xacro:boggie postfix="right" reflect="1"/>
+<xacro:boggie postfix="left" reflect="-1"/>
 <!-- end boggies -->
 <!-- wheels -->
-<xacro:macro name="wheel" params="side boggie reflect upsidedown">
+<xacro:macro name="wheel" params="side boggie reflect across rotation">
     <link name="wheel_axis_${side}_${boggie}">
         <visual>
@@ -142,11 +142,11 @@
         <xacro:wheel_inertial mass="1.0"/>
     </link>
-    <joint name="wheel_to_wheel_axis_${side}_${boggie}" type="fixed">
-        <origin rpy="0 0 ${reflect*3.14}" xyz="0 ${reflect*upsidedown*0.2} 0"/>
+    <joint name="boggie_${boggie}_to_wheel_axis_${side}_${boggie}" type="fixed">
+        <origin rpy="${reflect*across*-0.785398} 0 ${reflect*across*-3.14}" xyz="${reflect*-40.000E-03} ${across*-290.414E-03} -70.2315E-03"/>
         <parent link="boggie_${boggie}"/>
         <child link="wheel_axis_${side}_${boggie}"/>
     </joint>
-    <joint name="wheel_axis_to_wheel_holder_${side}_${boggie}" type="continuous">
-        <axis xyz="1 0 0"/>
+    <joint name="wheel_axis_${side}_${boggie}_to_wheel_${side}_${boggie}" type="continuous">
+        <axis xyz="${rotation} 0 0"/>
         <origin rpy="0 0 0" xyz="0 0 0"/>
         <parent link="wheel_axis_${side}_${boggie}"/>
@@ -154,8 +154,8 @@
     </joint>
 </xacro:macro>
-<xacro:wheel side="front" boggie="left" reflect="1" upsidedown="1" />
-<xacro:wheel side="front" boggie="right" reflect="-1" upsidedown="1" />
-<xacro:wheel side="back" boggie="left" reflect="1" upsidedown="-1" />
-<xacro:wheel side="back" boggie="right" reflect="-1" upsidedown="-1" />
+<xacro:wheel side="front" boggie="left" across="-1" reflect="1" rotation="1"/>
+<xacro:wheel side="front" boggie="right" across="1" reflect="1" rotation="-1"/>
+<xacro:wheel side="back" boggie="left" across="1" reflect="1" rotation="1"/>
+<xacro:wheel side="back" boggie="right" across="-1" reflect="1" rotation="-1"/>
 <!-- end wheels -->
 </robot>

Commit message: Modified CMakeLists. Fixed the inertial matrixes for the robot model. Disabled collisions for lighter Gazebo simulation until adding collision boxes.

File: urdf/jimmbot.xacro (robot description, xacro)
@@ -7,10 +7,10 @@
     <mass value="${mass}"/>
     <inertia
-              ixx="1"
-              ixy="1"
-              ixz="1"
-              iyy="1"
-              iyz="1"
-              izz="1" />
+      ixx="0.000001"
+      ixy="0"
+      ixz="0"
+      iyy="0.000001"
+      iyz="0"
+      izz="0.000001" />
   </inertial>
 </xacro:macro>
@@ -18,20 +18,12 @@
   <inertial>
     <mass value="${mass}"/>
-    <!-- <inertia
-              ixx="6.994E+08"
-              ixy="3.083E+05"
-              ixz="-2.746E+05"
-              iyy="1.202E+09"
-              iyz="-6.256E+05"
-              izz="1.446E+09" />
-  </inertial> -->
-  <inertia
-              ixx="5.78216276846"
-              ixy="0"
-              ixz="0"
-              iyy="10.4480713745"
-              iyz="0"
-              izz="12.8806369068" />
-  </inertial>
+    <inertia
+      ixx="0.578216276846"
+      ixy="0"
+      ixz="0"
+      iyy="1.04480713745"
+      iyz="0"
+      izz="1.28806369068" />
+    </inertial>
 </xacro:macro>
 <xacro:macro name="boggie_inertial" params="mass">
@@ -39,10 +31,10 @@
     <mass value="${mass}"/>
     <inertia
-              ixx="1.327E+07"
-              ixy="-1.417E+04"
-              ixz="-4.374E+05"
-              iyy="2.052E+08"
-              iyz="-1.830E+06"
-              izz="1.947E+08" />
+      ixx="0.260999632051"
+      ixy="0"
+      ixz="0"
+      iyy="0.0589854292796"
+      iyz="0"
+      izz="0.207161688318" />
   </inertial>
 </xacro:macro>
@@ -51,10 +43,10 @@
     <mass value="${mass}"/>
     <inertia
-              ixx="4.476E+04"
-              ixy="-1.834E+05"
-              ixz="-1.686E+05"
-              iyy="1.446E+06"
-              iyz="-2.198E+04"
-              izz="1.450E+06" />
+      ixx="1.664e-06"
+      ixy="0"
+      ixz="0"
+      iyy="4.0157e-05"
+      iyz="0"
+      izz="4.0157e-05" />
   </inertial>
 </xacro:macro>
@@ -63,10 +55,10 @@
     <mass value="${mass}"/>
     <inertia
-              ixx="4.654E+06"
-              ixy="-7.410E+06"
-              ixz="-6.730E+06"
-              iyy="5.291E+07"
-              iyz="-9.714E+05"
-              izz="5.309E+07" />
+      ixx="0.007139697375"
+      ixy="0"
+      ixz="0"
+      iyy="0.004079848688"
+      iyz="0"
+      izz="0.004079848688" />
   </inertial>
 </xacro:macro>
@@ -75,10 +67,22 @@
     <mass value="${mass}"/>
     <inertia
-              ixx="9.420E+04"
-              ixy="-1.785E-10"
-              ixz="-2.393E-06"
-              iyy="5.077E+06"
-              iyz="0.00"
-              izz="5.039E+06" />
+      ixx="0.00030833333333"
+      ixy="0"
+      ixz="0"
+      iyy="0.00478833333333"
+      iyz="0"
+      izz="0.00453333333333" />
+  </inertial>
+</xacro:macro>
+<xacro:macro name="differential_rod_inertial" params="mass">
+  <inertial>
+    <mass value="${mass}"/>
+    <inertia
+      ixx="2.39452259042e-07"
+      ixy="0"
+      ixz="0"
+      iyy="1.18596127489e-05"
+      iyz="0"
+      izz="1.20323211349e-05" />
   </inertial>
 </xacro:macro>
@@ -100,12 +104,11 @@
       <material name="silver"/>
     </visual>
-  <collision>
+  <!-- <collision>
     <origin rpy="0 0 0" xyz="0 0 0"/>
     <geometry>
         <mesh filename="package://jimmbot_description/meshes/chassis/chassis.stl" scale="0.001 0.001 0.001"/>
     </geometry>
-  </collision>
+  </collision> -->
   <xacro:chassis_inertial mass="40.0"/>
-  <!-- <xacro:zero_inertial mass="40"/> -->
 </link>
 <!-- end chassis -->
@@ -122,12 +125,11 @@
             <material name="silver"/>
         </visual>
-        <collision>
+        <!-- <collision>
             <origin rpy="0 0 0" xyz="0 0 0"/>
             <geometry>
                 <mesh filename="package://jimmbot_description/meshes/boggie/boggie.stl" scale="0.001 0.001 0.001"/>
             </geometry>
-        </collision>
-        <!-- <xacro:boggie_inertial mass="6.0"/> -->
-        <xacro:zero_inertial mass="6.0"/>
+        </collision> -->
+        <xacro:boggie_inertial mass="6.0"/>
     </link>
     <joint name="boggie_${postfix}_front_rods_to_boggie_${postfix}" type="fixed">
@@ -141,5 +143,5 @@
         <child link="boggie_${postfix}_back_rods"/>
     </joint>
-    <joint name="chassis_to_boggie_${postfix}" type="revolute">
+    <joint name="chassis_to_boggie_${postfix}" type="fixed">
         <axis xyz="${reflect*-1} 0 0"/>
         <limit effort="1000.0" lower="-0.523599" upper="0.523599" velocity="50"/>
@@ -164,12 +166,11 @@
             <material name="silver"/>
         </visual>
-        <collision>
+        <!-- <collision>
             <origin rpy="0 0 0" xyz="0 0 0"/>
             <geometry>
                 <mesh filename="package://jimmbot_description/meshes/differential/differential.stl" scale="0.001 0.001 0.001"/>
             </geometry>
-        </collision>
-        <!-- <xacro:differential_inertial mass="0.8"/> -->
-        <xacro:zero_inertial mass="0.8"/>
+        </collision> -->
+        <xacro:differential_inertial mass="0.8"/>
     </link>
     <joint name="differential_${postfix}_to_differential_left_${postfix}" type="fixed">
@@ -183,5 +184,5 @@
         <child link="differential_right_${postfix}"/>
     </joint>
-    <joint name="chassis_to_differential_${postfix}" type="revolute">
+    <joint name="chassis_to_differential_${postfix}" type="fixed">
         <axis xyz="0 0 -1"/>
         <limit effort="1000.0" lower="-0.523599" upper="0.523599" velocity="50"/>
@@ -197,6 +198,6 @@
 <xacro:macro name="differential_rod" params="postfix boggie reflect">
     <link name="differential_rod_differential_${postfix}_${boggie}" />
-    <link name="differential_rod_boggie_${postfix}_${boggie}" />
-    <!-- <link name="differential_rod_${postfix}_${boggie}">
+    <!-- <link name="differential_rod_boggie_${postfix}_${boggie}" /> -->
+    <link name="differential_rod_${postfix}_${boggie}">
         <visual>
             <origin rpy="0 0 0" xyz="0 0 0"/>
@@ -206,42 +207,27 @@
             <material name="silver"/>
         </visual>
-        <collision>
+        <!-- <collision>
             <origin rpy="0 0 0" xyz="0 0 0"/>
             <geometry>
                 <mesh filename="package://jimmbot_description/meshes/differential/differential_rod.stl" scale="0.01 0.01 0.01"/>
             </geometry>
-        </collision>
-        <xacro:differential_inertial mass="0.8"/>
-    </link> -->
-    <!-- <joint name="differential_rod_${postfix}_${boggie}_to_differential_rod_boggie_${postfix}_${boggie}" type="fixed">
+        </collision> -->
+        <xacro:differential_rod_inertial mass="0.4"/>
+    </link>
+    <joint name="differential_rod_${postfix}_${boggie}_to_differential_rod_differential_${postfix}_${boggie}" type="fixed">
         <origin rpy="0 0 0" xyz="-82E-03 0 0"/>
-        <parent link="differential_rod_${postfix}_${boggie}"/>
-        <child link="differential_rod_boggie_${postfix}_${boggie}"/>
-    </joint>
-    <joint name="differential_rod_${postfix}_${boggie}_to_differential_rod_differential_${postfix}_${boggie}" type="fixed">
-        <origin rpy="0 0 0" xyz="82E-03 0 0"/>
         <parent link="differential_rod_differential_${postfix}_${boggie}"/>
         <child link="differential_rod_${postfix}_${boggie}"/>
-    </joint> -->
-    <joint name="differential_rod_boggie_${postfix}_${boggie}_to_boggie_${boggie}" type="continuous">
-        <origin rpy="0 0.087266 ${reflect*-0.453786}" xyz="${reflect*0} 0 50E-03"/>
-        <parent link="boggie_${boggie}_${postfix}_rods"/>
-        <child link="differential_rod_boggie_${postfix}_${boggie}"/>
-    </joint>
-    <joint name="differential_rod_differential_${postfix}_${boggie}_to_differential_${boggie}_${postfix}" type="continuous">
-        <origin rpy="0 0.087266 ${reflect*0.453786}" xyz="${reflect*0} 0 50E-03"/>
+    </joint>
+    <joint name="differential_rod_differential_${postfix}_${boggie}_to_differential_${boggie}_${postfix}" type="fixed">
+        <origin rpy="0 0.087266 ${reflect+0.4537}" xyz="0 0 17E-03"/>
         <parent link="differential_${boggie}_${postfix}"/>
         <child link="differential_rod_differential_${postfix}_${boggie}"/>
     </joint>
-    <!-- <joint name="differential_rod_boggie_${postfix}_${boggie}_to_differential_rod_differential_${postfix}_${boggie}" type="fixed">
-        <origin rpy="0 0 0" xyz="0 0 0"/>
-        <parent link="differential_rod_differential_${postfix}_${boggie}"/>
-        <child link="differential_rod_boggie_${postfix}_${boggie}"/>
-    </joint> -->
-</xacro:macro>
-<xacro:differential_rod postfix="front" boggie="right" reflect="1"/>
-<xacro:differential_rod postfix="front" boggie="left" reflect="-1"/>
-<xacro:differential_rod postfix="back" boggie="right" reflect="1"/>
-<!-- <xacro:differential_rod postfix="front" boggie="left" reflect="-1"/> -->
+</xacro:macro>
+<xacro:differential_rod postfix="front" boggie="right" reflect="-1.57"/>
+<xacro:differential_rod postfix="front" boggie="left" reflect="-2.4774"/>
+<xacro:differential_rod postfix="back" boggie="right" reflect="-1.57"/>
+<xacro:differential_rod postfix="back" boggie="left" reflect="-2.4774"/>
 <!-- end differential_rod -->
 <!-- wheels -->
@@ -255,29 +241,27 @@
             <material name="silver"/>
         </visual>
+        <!-- <collision>
+            <origin rpy="0 0 0" xyz="0 0 0"/>
+            <geometry>
+                <mesh filename="package://jimmbot_description/meshes/wheel/wheel_axis.stl" scale="0.001 0.001 0.001"/>
+            </geometry>
+        </collision> -->
+        <xacro:wheel_axis_inertial mass="0.039"/>
+    </link>
+    <link name="wheel_${side}_${boggie}">
+        <visual>
+            <origin rpy="0 0 0" xyz="0 0 0"/>
+            <geometry>
+                <mesh filename="package://jimmbot_description/meshes/wheel/wheel.stl" scale="0.001 0.001 0.001"/>
+            </geometry>
+            <material name="silver"/>
+        </visual>
         <collision>
             <origin rpy="0 0 0" xyz="0 0 0"/>
             <geometry>
-                <mesh filename="package://jimmbot_description/meshes/wheel/wheel_axis.stl" scale="0.001 0.001 0.001"/>
+                <mesh filename="package://jimmbot_description/meshes/wheel/wheel.stl" scale="0.001 0.001 0.001"/>
             </geometry>
         </collision>
-        <!-- <xacro:wheel_axis_inertial mass="0.039"/> -->
-        <xacro:zero_inertial mass="0.039"/>
-    </link>
-    <link name="wheel_${side}_${boggie}">
-        <visual>
-            <origin rpy="0 0 0" xyz="0 0 0"/>
-            <geometry>
-                <mesh filename="package://jimmbot_description/meshes/wheel/wheel.stl" scale="0.001 0.001 0.001"/>
-            </geometry>
-            <material name="silver"/>
-        </visual>
-        <collision>
-            <origin rpy="0 0 0" xyz="0 0 0"/>
-            <geometry>
-                <mesh filename="package://jimmbot_description/meshes/wheel/wheel.stl" scale="0.001 0.001 0.001"/>
-            </geometry>
-        </collision>
-        <!-- <xacro:wheel_inertial mass="1.0"/> -->
-        <xacro:zero_inertial mass="1.0"/>
+        <xacro:wheel_inertial mass="1.7"/>
     </link>
     <joint name="boggie_${boggie}_to_wheel_axis_${side}_${boggie}" type="fixed">

Commit message: Added kinect, and ydlidar meshes. Also updated the xacro URDF file.

File: urdf/jimmbot.xacro (robot description, xacro)
@@ -37,4 +37,28 @@
       iyz="0"
       izz="0.207161688318" />
+  </inertial>
+</xacro:macro>
+<xacro:macro name="lidar_inertial_base" params="mass">
+  <inertial>
+    <mass value="${mass}"/>
+    <inertia
+      ixx="6.7885E-05"
+      ixy="-1.3987E-07"
+      ixz="-8.1554E-07"
+      iyy="0.00013173"
+      iyz="-9.0932E-08"
+      izz="7.1972E-05" />
+  </inertial>
+</xacro:macro>
+<xacro:macro name="lidar_inertial_frame" params="mass">
+  <inertial>
+    <mass value="${mass}"/>
+    <inertia
+      ixx="8.9194E-05"
+      ixy="1.8116E-07"
+      ixz="3.6435E-08"
+      iyy="0.00018279"
+      iyz="2.423E-07"
+      izz="0.00011103" />
   </inertial>
 </xacro:macro>
@@ -113,4 +137,190 @@
 </link>
 <!-- end chassis -->
+<!-- imu -->
+<xacro:macro name="imu">
+    <link name="imu_base">
+        <visual>
+            <origin rpy="0 0 0" xyz="0 0 0"/>
+            <geometry>
+                <box size="0.1 0.1 0.1" />
+            </geometry>
+            <material name="silver"/>
+        </visual>
+        <collision>
+            <origin rpy="0 0 0" xyz="0 0 0"/>
+            <geometry>
+                <box size="0.01 0.2 0.01" />
+            </geometry>
+        </collision>
+        <xacro:lidar_inertial_base mass="0.15717"/>
+    </link>
+    <gazebo reference="imu_base">
+      <gravity>true</gravity>
+      <sensor name="imu_sensor" type="imu">
+        <always_on>true</always_on>
+        <update_rate>100</update_rate>
+        <visualize>true</visualize>
+        <topic>__default_topic__</topic>
+        <plugin filename="libgazebo_ros_imu_sensor.so" name="imu_plugin">
+          <topicName>imu</topicName>
+          <bodyName>imu_base</bodyName>
+          <updateRateHZ>10.0</updateRateHZ>
+          <gaussianNoise>0.0</gaussianNoise>
+          <xyzOffset>0 0 0</xyzOffset>
+          <rpyOffset>0 0 0</rpyOffset>
+          <frameName>imu_base</frameName>
+          <initialOrientationAsReference>false</initialOrientationAsReference>
+        </plugin>
+        <pose>0 0 0 0 0 0</pose>
+      </sensor>
+    </gazebo>
+    <joint name="chassis_to_imu" type="fixed">
+        <axis xyz="0 0 0"/>
+        <origin rpy="0 0 0" xyz="0 0 0"/>
+        <parent link="chassis"/>
+        <child link="imu_base"/>
+    </joint>
+</xacro:macro>
+<xacro:imu />
+<!-- end imu -->
+<!-- lidar -->
+<xacro:macro name="lidar">
+    <link name="lidar_base">
+        <visual>
+            <origin rpy="0 0 0" xyz="0 0 0"/>
+            <geometry>
+                <mesh filename="package://jimmbot_description/meshes/ydlidar/ydlidar.dae" />
+            </geometry>
+            <material name="lidar"/>
+        </visual>
+        <collision>
+            <origin rpy="0 0 0" xyz="0 0 0"/>
+            <geometry>
+                <mesh filename="package://jimmbot_description/meshes/ydlidar/ydlidar.dae" />
+            </geometry>
+        </collision>
+        <xacro:lidar_inertial_base mass="0.15717"/>
+    </link>
+    <link name="lidar_frame">
+        <xacro:lidar_inertial_frame mass="0.25482"/>
+    </link>
+    <joint name="laser_joint" type="fixed">
+        <origin rpy="0 0 0" xyz="0 0 0.03172" />
+        <parent link="lidar_base" />
+        <child link="lidar_frame" />
+        <axis xyz="0 0 0" />
+    </joint>
+    <gazebo reference="imu_base">
+      <gravity>true</gravity>
+      <sensor type="ray" name="sensor">
+        <!-- Enable visualization to see the rays in the GUI -->
+        <visualize>true</visualize>
+        <!-- Set the update rate of the sensor -->
+        <update_rate>10</update_rate>
+        <ray>
+          <!-- The scan element contains the horizontal and vertical beams.
+              We are leaving out the vertical beams for this tutorial. -->
+          <scan>
+            <!-- The horizontal beams -->
+            <horizontal>
+              <!-- The velodyne has 32 beams(samples) -->
+              <samples>360</samples>
+              <!-- Resolution is multiplied by samples to determine number of
+                  simulated beams vs interpolated beams. See:
+                  http://sdformat.org/spec?ver=1.6&elem=sensor#horizontal_resolution
+                  -->
+              <resolution>1</resolution>
+              <!-- Minimum angle in radians -->
+              <min_angle>-6.28319</min_angle>
+              <!-- Maximum angle in radians -->
+              <max_angle>6.28319</max_angle>
+            </horizontal>
+          </scan>
+          <!-- Range defines characteristics of an individual beam -->
+          <range>
+            <!-- Minimum distance of the beam -->
+            <min>0.05</min>
+            <!-- Maximum distance of the beam -->
+            <max>15</max>
+            <!-- Linear resolution of the beam -->
+            <resolution>0.02</resolution>
+          </range>
+        </ray>
+      </sensor>
+    </gazebo>
+    <joint name="chassis_to_lidar" type="fixed">
+        <axis xyz="0 0 0"/>
+        <origin rpy="0 0 0" xyz="0 0 0.15"/>
+        <parent link="chassis"/>
+        <child link="lidar_base"/>
+    </joint>
+</xacro:macro>
+<xacro:lidar />
+<!-- end lidar -->
+<!-- kinect -->
+<xacro:macro name="kinect" params="postfix reflect">
+    <link name="kinect_${postfix}">
+        <visual>
+            <origin rpy="0 0 0" xyz="0 0 0"/>
+            <geometry>
+                <mesh filename="package://jimmbot_description/meshes/kinect/kinect.dae" />
+            </geometry>
+            <material name="silver"/>
+        </visual>
+        <!-- <collision>
+            <origin rpy="0 0 0" xyz="0 0 0"/>
+            <geometry>
+                <mesh filename="package://jimmbot_description/meshes/boggie/boggie.stl" scale="0.001 0.001 0.001"/>
+            </geometry>
+        </collision> -->
+        <!-- <xacro:kinect_inertial mass="6.0"/> -->
+    </link>
+    <gazebo reference="kinect_${postfix}">
+      <sensor type="depth" name="${postfix}">
+        <always_on>true</always_on>
+        <update_rate>20.0</update_rate>
+        <camera>
+          <horizontal_fov>${60.0*3.14/180.0}</horizontal_fov>
+          <image>
+            <format>R8G8B8</format>
+            <width>640</width>
+            <height>480</height>
+          </image>
+          <clip>
+            <near>0.05</near>
+            <far>8.0</far>
+          </clip>
+        </camera>
+        <plugin name="kinect_${postfix}_controller" filename="libgazebo_ros_openni_kinect.so">
+          <cameraName>${postfix}</cameraName>
+          <alwaysOn>true</alwaysOn>
+          <updateRate>10</updateRate>
+          <imageTopicName>rgb/image_raw</imageTopicName>
+          <depthImageTopicName>depth/image_raw</depthImageTopicName>
+          <pointCloudTopicName>depth/points</pointCloudTopicName>
+          <cameraInfoTopicName>rgb/camera_info</cameraInfoTopicName>
+          <depthImageCameraInfoTopicName>depth/camera_info</depthImageCameraInfoTopicName>
+          <frameName>kinect_${postfix}</frameName>
+          <baseline>0.1</baseline>
+          <distortion_k1>0.0</distortion_k1>
+          <distortion_k2>0.0</distortion_k2>
+          <distortion_k3>0.0</distortion_k3>
+          <distortion_t1>0.0</distortion_t1>
+          <distortion_t2>0.0</distortion_t2>
+          <pointCloudCutoff>0.4</pointCloudCutoff>
+          <robotNamespace>/</robotNamespace>
+        </plugin>
+      </sensor>
+    </gazebo>
+    <joint name="chassis_to_kinect_${postfix}" type="fixed">
+        <axis xyz="${reflect*-1} 0 0"/>
+        <origin rpy="0.523599 0 ${reflect*1.57}" xyz="${reflect*0.25} 0 0.11"/>
+        <parent link="chassis"/>
+        <child link="kinect_${postfix}"/>
+    </joint>
+</xacro:macro>
+<xacro:kinect postfix="front" reflect="1"/>
+<xacro:kinect postfix="back" reflect="-1"/>
+<!-- end kinect -->
 <!-- boggies -->
 <xacro:macro name="boggie" params="postfix reflect">
@@ -298,8 +508,8 @@
 this turn off, and implemented hardware interface read() and write() functions, will publish speeds from real hardware
 -->
-<gazebo>
+<!-- <gazebo>
   <plugin name="gazebo_ros_control" filename= "libgazebo_ros_control.so">
    <robotNamespace>/</robotNamespace>
   </plugin>
-</gazebo>
+</gazebo> -->
 </robot>

File: urdf/materials.xacro (robot description, xacro)
@@ -2,5 +2,8 @@
 <robot name="jimmbot" xmlns:xacro="http://www.ros.org/wiki/xacro" >
 <material name="silver">
-  <color rgba="0.700 0.700 0.700 1.000"/>
+  <color rgba="0.700 0.700 0.700 1.000" />
+</material>
+<material name="lidar">
+  <color rgba="0.64706 0.61961 0.58824 1" />
 </material>
 </robot>
