Commit message: Fix merge conflicts in xml.

File: urdf/jimmbot.gazebo.xacro (robot description, xacro)
@@ -2,5 +2,5 @@
 <robot name="jimmbot_simulation" xmlns:xacro="http://ros.org/wiki/xacro">
   <!-- Kinect front -->
-  <gazebo reference="kinect_front">
+  <gazebo reference="kinect_front_link">
     <sensor type="depth" name="front">
       <always_on>true</always_on>
@@ -39,5 +39,5 @@
   </gazebo>
   <!-- Kinect back -->
-  <gazebo reference="kinect_back">
+  <gazebo reference="kinect_back_link">
     <sensor type="depth" name="back">
       <always_on>true</always_on>

File: urdf/jimmbot.xacro (robot description, xacro)
@@ -136,47 +136,5 @@
     </joint>
     <link name="kinect_${postfix}_optical"/>
-<<<<<<< HEAD
     <joint name="chassis_to_kinect_${postfix}" type="fixed">
-=======
-    <!-- Transfer to gazebo xacro -->
-    <gazebo reference="kinect_${postfix}_link">
-      <sensor type="depth" name="${postfix}">
-        <always_on>true</always_on>
-        <update_rate>20.0</update_rate>
-        <camera>
-          <horizontal_fov>${60.0*3.14/180.0}</horizontal_fov>
-          <image>
-            <format>R8G8B8</format>
-            <width>640</width>
-            <height>480</height>
-          </image>
-          <clip>
-            <near>0.05</near>
-            <far>8.0</far>
-          </clip>
-        </camera>
-        <plugin name="kinect_${postfix}_controller" filename="libgazebo_ros_openni_kinect.so">
-          <cameraName>${postfix}</cameraName>
-          <alwaysOn>true</alwaysOn>
-          <updateRate>10</updateRate>
-          <imageTopicName>rgb/image_raw</imageTopicName>
-          <depthImageTopicName>depth/image_raw</depthImageTopicName>
-          <pointCloudTopicName>depth/points</pointCloudTopicName>
-          <cameraInfoTopicName>rgb/camera_info</cameraInfoTopicName>
-          <depthImageCameraInfoTopicName>depth/camera_info</depthImageCameraInfoTopicName>
-          <frameName>kinect_${postfix}_optical</frameName>
-          <baseline>0.1</baseline>
-          <distortion_k1>0.0</distortion_k1>
-          <distortion_k2>0.0</distortion_k2>
-          <distortion_k3>0.0</distortion_k3>
-          <distortion_t1>0.0</distortion_t1>
-          <distortion_t2>0.0</distortion_t2>
-          <pointCloudCutoff>0.4</pointCloudCutoff>
-          <robotNamespace>/</robotNamespace>
-        </plugin>
-      </sensor>
-    </gazebo>
-    <joint name="chassis_to_kinect_${postfix}_link" type="fixed">
->>>>>>> 578b3543b0f9ed2c718524d3e05bda4a321d6d62
         <origin rpy="0 0.523599 ${reflect*1.5708-1.5708}" xyz="${reflect*0.25} 0 0.11"/>
         <parent link="chassis"/>

Commit message: Added license in package. Changed position in description and changed kinect names, so we are same in simulation and real robot.

File: urdf/jimmbot.gazebo.xacro (robot description, xacro)
@@ -3,5 +3,5 @@
   <!-- Kinect front -->
   <gazebo reference="kinect_front_link">
-    <sensor type="depth" name="front">
+    <sensor type="depth" name="kinect_front">
       <always_on>true</always_on>
       <update_rate>20.0</update_rate>
@@ -19,8 +19,8 @@
       </camera>
       <plugin name="kinect_front_controller" filename="libgazebo_ros_openni_kinect.so">
-        <cameraName>front</cameraName>
+        <cameraName>kinect_front</cameraName>
         <alwaysOn>true</alwaysOn>
         <updateRate>10</updateRate>
-        <imageTopicName>rgb/image_raw</imageTopicName>
+        <imageTopicName>rgb/image_color</imageTopicName>
         <depthImageTopicName>depth/image_raw</depthImageTopicName>
         <pointCloudTopicName>depth/points</pointCloudTopicName>
@@ -40,5 +40,5 @@
   <!-- Kinect back -->
   <gazebo reference="kinect_back_link">
-    <sensor type="depth" name="back">
+    <sensor type="depth" name="kinect_back">
       <always_on>true</always_on>
       <update_rate>20.0</update_rate>
@@ -56,8 +56,8 @@
       </camera>
       <plugin name="kinect_back_controller" filename="libgazebo_ros_openni_kinect.so">
-        <cameraName>back</cameraName>
+        <cameraName>kinect_back</cameraName>
         <alwaysOn>true</alwaysOn>
         <updateRate>10</updateRate>
-        <imageTopicName>rgb/image_raw</imageTopicName>
+        <imageTopicName>rgb/image_color</imageTopicName>
         <depthImageTopicName>depth/image_raw</depthImageTopicName>
         <pointCloudTopicName>depth/points</pointCloudTopicName>

File: urdf/jimmbot.xacro (robot description, xacro)
@@ -247,5 +247,5 @@
     </joint>
     <joint name="differential_rod_differential_${postfix}_${boggie}_to_differential_${boggie}_${postfix}" type="fixed">
-        <origin rpy="0 0.087266 ${reflect+0.4537}" xyz="0 0 17E-03"/>
+        <origin rpy="0 0 ${reflect+0.4537}" xyz="0 0 17E-03"/>
         <parent link="differential_${boggie}_${postfix}"/>
         <child link="differential_rod_differential_${postfix}_${boggie}"/>

Commit message: Fixed some position problems in model. Also switching slowly from stl to dae, in order to have a better visualization of the robot. WIP: Chassis

File: urdf/jimmbot.gazebo.xacro (robot description, xacro)
@@ -124,4 +124,54 @@
     </sensor>
   </gazebo>
+<!-- @todo Check if this or gazebo_imu is better -->
+  <!-- <gazebo>
+    <plugin name="imu_base" filename="libhector_gazebo_ros_imu.so">
+      <serviceName>/imu/calibrate</serviceName>
+      <updateRate>200.0</updateRate>
+      <bodyName>imu_base</bodyName>
+      <frameId>imu_base</frameId>
+      <topicName>imu</topicName>
+      <rpyOffset>0 0 0</rpyOffset>
+      <xyzOffset>0 0 0</xyzOffset>
+      <gaussianNoise>0.00000001</gaussianNoise>
+      <accelDrift>0.00000001 0.00000001 0.00000001</accelDrift>
+      <accelDriftFrequency>0.00000001 0.00000001 0.00000001</accelDriftFrequency>
+      <accelGaussianNoise>0.00000001 0.00000001 0.00000001</accelGaussianNoise>
+      <rateDrift>0.0 0.0 0.0</rateDrift>
+      <rateDriftFrequency>0.0 0.0 0.0</rateDriftFrequency>
+      <rateGaussianNoise>0.0 0.0 0.0</rateGaussianNoise>
+      <headingDrift>0.0 0.0 0.0</headingDrift>
+      <headingDriftFrequency>0.0 0.0 0.0</headingDriftFrequency>
+      <headingGaussianNoise>0.0 0.0 0.0</headingGaussianNoise>
+    </plugin>
+  </gazebo> -->
+  <gazebo>
+    <plugin name="gps_sensor_front" filename="libhector_gazebo_ros_gps.so">
+        <alwayson>true</alwayson>
+        <updaterate>10.0</updaterate>
+        <bodyname>gps_front_base</bodyname>
+        <frameId>gps_front_base</frameId>
+        <topicName>gps/fix_front</topicName>
+        <velocityTopicName>gps/fix_front_velocity</velocityTopicName>
+        <drift>0.001 0.001 0.001</drift>
+        <gaussianNoise>0.05 0.05 0.05</gaussianNoise>
+        <velocityDrift>0.001 0.001 0.001</velocityDrift>
+        <velocityGaussianNoise>0.5 0.5 0.5</velocityGaussianNoise>
+    </plugin>
+  </gazebo>
+  <gazebo>
+    <plugin name="gps_sensor_back" filename="libhector_gazebo_ros_gps.so">
+        <alwayson>true</alwayson>
+        <updaterate>10.0</updaterate>
+        <bodyname>gps_back_base</bodyname>
+        <frameId>gps_back_base</frameId>
+        <topicName>/gps/fix_back</topicName>
+        <velocityTopicName>/gps/fix_back_velocity</velocityTopicName>
+        <drift>0.001 0.001 0.001</drift>
+        <gaussianNoise>0.05 0.05 0.05</gaussianNoise>
+        <velocityDrift>0.001 0.001 0.001</velocityDrift>
+        <velocityGaussianNoise>0.5 0.5 0.5</velocityGaussianNoise>
+    </plugin>
+  </gazebo>
   <gazebo>
     <plugin name="gazebo_ros_control" filename= "libgazebo_ros_control.so">

File: urdf/jimmbot.xacro (robot description, xacro)
@@ -54,4 +54,56 @@
 <xacro:imu />
 <!-- end imu -->
+<!-- gps -->
+<xacro:macro name="gps" params="postfix reflect">
+    <link name="gps_${postfix}_base">
+        <visual>
+            <origin rpy="0 0 0" xyz="0 0 0"/>
+            <geometry>
+                <mesh filename="package://jimmbot_description/meshes/gps/linx_gps.dae" />
+            </geometry>
+        </visual>
+        <collision>
+            <origin rpy="0 0 0" xyz="0 0 0"/>
+            <geometry>
+                <mesh filename="package://jimmbot_description/meshes/gps/linx_gps.dae" />
+            </geometry>
+        </collision>
+        <!-- <xacro:gps_inertial mass="0.58"/> -->
+    </link>
+    <joint name="chassis_to_gps_${postfix}" type="fixed">
+        <origin rpy="1.5708 0 ${reflect*1.5708-1.5708}" xyz="${reflect*0.1} ${reflect*-0.1} 0.117"/>
+        <parent link="chassis"/>
+        <child link="gps_${postfix}_base"/>
+    </joint>
+</xacro:macro>
+<xacro:gps postfix="front" reflect="1"/>
+<xacro:gps postfix="back" reflect="-1"/>
+<!-- end gps -->
+<!-- wifi_antenna -->
+<xacro:macro name="wifi_antenna" params="postfix reflect">
+  <link name="wifi_antenna_${postfix}_base">
+    <visual>
+      <origin rpy="0 0 0" xyz="0 0 0"/>
+      <geometry>
+        <mesh filename="package://jimmbot_description/meshes/wifi_antenna/wifi_antenna.dae" />
+      </geometry>
+    </visual>
+    <collision>
+      <origin rpy="0 0 0" xyz="0 0 0"/>
+      <geometry>
+        <mesh filename="package://jimmbot_description/meshes/wifi_antenna/wifi_antenna.dae" />
+      </geometry>
+    </collision>
+    <!-- <xacro:wifi_antenna_inertial mass="0.58"/> -->
+  </link>
+  <joint name="chassis_to_wifi_antenna_${postfix}" type="fixed">
+    <origin rpy="1.5708 0 ${reflect*1.5708-1.5708}" xyz="${reflect*-0.06} ${reflect*0.1} 0.13"/>
+    <parent link="chassis"/>
+    <child link="wifi_antenna_${postfix}_base"/>
+  </joint>
+</xacro:macro>
+<xacro:wifi_antenna postfix="front" reflect="1"/>
+<xacro:wifi_antenna postfix="back" reflect="-1"/>
+<!-- end wifi_antenna -->
 <!-- lidar -->
 <xacro:macro name="lidar">
@@ -117,5 +169,5 @@
     <link name="kinect_${postfix}_link">
         <visual>
-            <origin rpy="0 0 1.57" xyz="0 0 0"/>
+            <origin rpy="0 0 1.5708" xyz="0 0 0"/>
             <geometry>
                 <mesh filename="package://jimmbot_description/meshes/kinect/kinect.dae" />
@@ -153,11 +205,11 @@
             <origin rpy="0 0 0" xyz="0 0 0"/>
             <geometry>
-                <mesh filename="package://jimmbot_description/meshes/boggie/boggie.stl" scale="0.001 0.001 0.001"/>
-            </geometry>
-        </visual>
-        <collision>
-            <origin rpy="0 0 0" xyz="0 0 0"/>
-            <geometry>
-                <mesh filename="package://jimmbot_description/meshes/boggie/boggie.stl" scale="0.001 0.001 0.001"/>
+                <mesh filename="package://jimmbot_description/meshes/boggie/boggie.dae" scale="0.001 0.001 0.001"/>
+            </geometry>
+        </visual>
+        <collision>
+            <origin rpy="0 0 0" xyz="0 0 0"/>
+            <geometry>
+                <mesh filename="package://jimmbot_description/meshes/boggie/boggie.dae" scale="0.001 0.001 0.001"/>
             </geometry>
         </collision>
@@ -175,5 +227,5 @@
     </joint>
     <joint name="chassis_to_boggie_${postfix}" type="fixed">
-        <origin rpy="0 0 ${reflect*1.57}" xyz="${reflect*-1.45758E-03} ${reflect*-201.552E-03} -19.8088E-03"/>
+        <origin rpy="0 0 ${reflect*1.5708}" xyz="${reflect*-1.45758E-03} ${reflect*-201.552E-03} -19.8088E-03"/>
         <parent link="chassis"/>
         <child link="boggie_${postfix}"/>
@@ -214,5 +266,5 @@
     <joint name="chassis_to_differential_${postfix}" type="fixed">
         <limit effort="1000.0" lower="-0.523599" upper="0.523599" velocity="50"/>
-        <origin rpy="0 0 ${reflect*1.57}" xyz="${reflect*147.5E-03} 0 147.0E-03"/>
+        <origin rpy="0 0 ${reflect*1.5708}" xyz="${reflect*147.5E-03} 0 147.0E-03"/>
         <parent link="chassis"/>
         <child link="differential_${postfix}"/>
@@ -252,7 +304,7 @@
     </joint>
 </xacro:macro>
-<xacro:differential_rod postfix="front" boggie="right" reflect="-1.57"/>
+<xacro:differential_rod postfix="front" boggie="right" reflect="-1.5708"/>
 <xacro:differential_rod postfix="front" boggie="left" reflect="-2.4774"/>
-<xacro:differential_rod postfix="back" boggie="right" reflect="-1.57"/>
+<xacro:differential_rod postfix="back" boggie="right" reflect="-1.5708"/>
 <xacro:differential_rod postfix="back" boggie="left" reflect="-2.4774"/>
 <!-- end differential_rod -->
@@ -263,11 +315,11 @@
             <origin rpy="0 0 0" xyz="0 0 0"/>
             <geometry>
-                <mesh filename="package://jimmbot_description/meshes/wheel/wheel_axis.stl" scale="0.001 0.001 0.001"/>
-            </geometry>
-        </visual>
-        <collision>
-            <origin rpy="0 0 0" xyz="0 0 0"/>
-            <geometry>
-                <mesh filename="package://jimmbot_description/meshes/wheel/wheel_axis.stl" scale="0.001 0.001 0.001"/>
+                <mesh filename="package://jimmbot_description/meshes/wheel/wheel_axis.dae" scale="0.001 0.001 0.001"/>
+            </geometry>
+        </visual>
+        <collision>
+            <origin rpy="0 0 0" xyz="0 0 0"/>
+            <geometry>
+                <mesh filename="package://jimmbot_description/meshes/wheel/wheel_axis.dae" scale="0.001 0.001 0.001"/>
             </geometry>
         </collision>
@@ -278,5 +330,5 @@
             <origin rpy="0 0 0" xyz="0 0 0"/>
             <geometry>
-                <mesh filename="package://jimmbot_description/meshes/wheel/wheel.stl" scale="0.001 0.001 0.001"/>
+                <mesh filename="package://jimmbot_description/meshes/wheel/wheel.dae" scale="0.001 0.001 0.001"/>
             </geometry>
         </visual>
@@ -290,5 +342,5 @@
     </link>
     <joint name="boggie_${boggie}_to_wheel_axis_${side}_${boggie}" type="fixed">
-        <origin rpy="${reflect*across*-0.785398} 0 ${reflect*across*-3.14}" xyz="${reflect*-40.000E-03} ${across*-290.414E-03} -70.2315E-03"/>
+        <origin rpy="${reflect*across*-0.785398} 0 ${reflect*across*-3.14159}" xyz="${reflect*-40.000E-03} ${across*-290.414E-03} -70.2315E-03"/>
         <parent link="boggie_${boggie}"/>
         <child link="wheel_axis_${side}_${boggie}"/>
