Commit message: Add cpp17 compile option and fixed indentation. Also added changed some noise and position parameters.

File: urdf/jimmbot.gazebo.xacro (robot description, xacro)
@@ -86,7 +86,8 @@
         <bodyName>imu_base</bodyName>
         <updateRateHZ>50.0</updateRateHZ>
-        <gaussianNoise>0.0</gaussianNoise>
+        <gaussianNoise>0.05</gaussianNoise>
         <xyzOffset>0 0 0</xyzOffset>
         <rpyOffset>0 0 0</rpyOffset>
+        <yawOffset>1.5708</yawOffset>
         <frameName>imu_base</frameName>
         <initialOrientationAsReference>false</initialOrientationAsReference>
@@ -149,5 +150,5 @@
     <plugin name="gps_sensor_front" filename="libhector_gazebo_ros_gps.so">
         <alwayson>true</alwayson>
-        <updaterate>10.0</updaterate>
+        <updaterate>50.0</updaterate>
         <bodyname>gps_front_base</bodyname>
         <frameId>gps_front_base</frameId>
@@ -163,5 +164,5 @@
     <plugin name="gps_sensor_back" filename="libhector_gazebo_ros_gps.so">
         <alwayson>true</alwayson>
-        <updaterate>10.0</updaterate>
+        <updaterate>50.0</updaterate>
         <bodyname>gps_back_base</bodyname>
         <frameId>gps_back_base</frameId>

File: urdf/jimmbot.xacro (robot description, xacro)
@@ -15,11 +15,11 @@
     <origin rpy="0 0 0" xyz="0 0 0"/>
     <geometry>
-        <mesh filename="package://jimmbot_description/meshes/chassis/chassis.stl" scale="0.001 0.001 0.001"/>
-      </geometry>
-    </visual>
+      <mesh filename="package://jimmbot_description/meshes/chassis/chassis.stl" scale="0.001 0.001 0.001"/>
+    </geometry>
+  </visual>
   <collision>
     <origin rpy="0 0 0" xyz="0 0 0"/>
     <geometry>
-        <mesh filename="package://jimmbot_description/meshes/chassis/chassis.stl" scale="0.001 0.001 0.001"/>
+      <mesh filename="package://jimmbot_description/meshes/chassis/chassis.stl" scale="0.001 0.001 0.001"/>
     </geometry>
   </collision>
@@ -30,25 +30,25 @@
 <!-- imu -->
 <xacro:macro name="imu">
-    <link name="imu_base">
-        <visual>
-            <origin rpy="0 0 0" xyz="0 0 0"/>
-            <geometry>
-                <box size="0.037 0.052 0.035" />
-            </geometry>
-        </visual>
-        <!-- IMU is inside chassis, no need for collision, chassis collision will handle all inside the chassis -->
-        <!-- <collision>
-            <origin rpy="0 0 0" xyz="0 0 0"/>
-            <geometry>
-                <box size="0.037 0.052 0.035" />
-            </geometry>
-        </collision>
-        <xacro:lidar_inertial_base mass="0.15717"/> -->
-    </link>
-    <joint name="chassis_to_imu" type="fixed">
-        <origin rpy="0 0 0" xyz="0 0 0"/>
-        <parent link="chassis"/>
-        <child link="imu_base"/>
-    </joint>
+  <link name="imu_base">
+    <visual>
+      <origin rpy="0 0 0" xyz="0 0 0"/>
+      <geometry>
+        <box size="0.037 0.052 0.035" />
+      </geometry>
+    </visual>
+    <!-- IMU is inside chassis, no need for collision, chassis collision will handle all inside the chassis -->
+    <!-- <collision>
+      <origin rpy="0 0 0" xyz="0 0 0"/>
+      <geometry>
+        <box size="0.037 0.052 0.035" />
+      </geometry>
+    </collision>
+    <xacro:lidar_inertial_base mass="0.15717"/> -->
+  </link>
+  <joint name="chassis_to_imu" type="fixed">
+    <origin rpy="0 0 0" xyz="0 0 0"/>
+    <parent link="chassis"/>
+    <child link="imu_base"/>
+  </joint>
 </xacro:macro>
 <xacro:imu />
@@ -56,24 +56,24 @@
 <!-- gps -->
 <xacro:macro name="gps" params="postfix reflect">
-    <link name="gps_${postfix}_base">
-        <visual>
-            <origin rpy="0 0 0" xyz="0 0 0"/>
-            <geometry>
-                <mesh filename="package://jimmbot_description/meshes/gps/linx_gps.dae" />
-            </geometry>
-        </visual>
-        <collision>
-            <origin rpy="0 0 0" xyz="0 0 0"/>
-            <geometry>
-                <mesh filename="package://jimmbot_description/meshes/gps/linx_gps.dae" />
-            </geometry>
-        </collision>
-        <!-- <xacro:gps_inertial mass="0.58"/> -->
-    </link>
-    <joint name="chassis_to_gps_${postfix}" type="fixed">
-        <origin rpy="1.5708 0 ${reflect*1.5708-1.5708}" xyz="${reflect*0.1} ${reflect*-0.1} 0.117"/>
-        <parent link="chassis"/>
-        <child link="gps_${postfix}_base"/>
-    </joint>
+  <link name="gps_${postfix}_base">
+    <visual>
+      <origin rpy="0 0 0" xyz="0 0 0"/>
+      <geometry>
+        <mesh filename="package://jimmbot_description/meshes/gps/linx_gps.dae" />
+      </geometry>
+    </visual>
+    <collision>
+      <origin rpy="0 0 0" xyz="0 0 0"/>
+      <geometry>
+        <mesh filename="package://jimmbot_description/meshes/gps/linx_gps.dae" />
+      </geometry>
+    </collision>
+    <!-- <xacro:gps_inertial mass="0.58"/> -->
+  </link>
+  <joint name="chassis_to_gps_${postfix}" type="fixed">
+    <origin rpy="1.5708 0 ${reflect*1.5708-1.5708}" xyz="${reflect*0.1} ${reflect*-0.1} 0.117"/>
+    <parent link="chassis"/>
+    <child link="gps_${postfix}_base"/>
+  </joint>
 </xacro:macro>
 <xacro:gps postfix="front" reflect="1"/>
@@ -108,33 +108,32 @@
 <!-- lidar -->
 <xacro:macro name="lidar">
-    <link name="lidar_base">
-        <visual>
-            <origin rpy="0 0 0" xyz="0 0 0"/>
-            <geometry>
-                <mesh filename="package://jimmbot_description/meshes/ydlidar/ydlidar.dae" />
-            </geometry>
-        </visual>
-        <collision>
-            <origin rpy="0 0 0" xyz="0 0 0"/>
-            <geometry>
-                <mesh filename="package://jimmbot_description/meshes/ydlidar/ydlidar.dae" />
-            </geometry>
-        </collision>
-        <xacro:lidar_inertial_base mass="0.15717"/>
-    </link>
-    <link name="lidar_frame">
-        <xacro:lidar_inertial_frame mass="0.25482"/>
-    </link>
-    <joint name="laser_joint" type="fixed">
-        <origin rpy="0 0 0" xyz="0 0 0.03172" />
-        <parent link="lidar_base" />
-        <child link="lidar_frame" />
-        <axis xyz="0 0 0" />
-    </joint>
-    <joint name="chassis_to_lidar" type="fixed">
-        <origin rpy="0 0 0" xyz="0 0 0.060"/>
-        <parent link="lidar_mount"/>
-        <child link="lidar_base"/>
-    </joint>
+  <link name="lidar_base">
+    <visual>
+      <origin rpy="0 0 0" xyz="0 0 0"/>
+      <geometry>
+        <mesh filename="package://jimmbot_description/meshes/ydlidar/ydlidar.dae" />
+      </geometry>
+    </visual>
+    <collision>
+      <origin rpy="0 0 0" xyz="0 0 0"/>
+      <geometry>
+        <mesh filename="package://jimmbot_description/meshes/ydlidar/ydlidar.dae" />
+      </geometry>
+    </collision>
+    <xacro:lidar_inertial_base mass="0.15717"/>
+  </link>
+  <link name="lidar_frame">
+    <xacro:lidar_inertial_frame mass="0.25482"/>
+  </link>
+  <joint name="laser_joint" type="fixed">
+    <origin rpy="0 0 0" xyz="0 0 0.03172" />
+    <parent link="lidar_base" />
+    <child link="lidar_frame" />
+  </joint>
+  <joint name="chassis_to_lidar" type="fixed">
+    <origin rpy="0 0 0" xyz="0 0 0.060"/>
+    <parent link="lidar_mount"/>
+    <child link="lidar_base"/>
+  </joint>
 </xacro:macro>
 <xacro:lidar />
@@ -142,24 +141,24 @@
 <!-- lidar mount -->
 <xacro:macro name="lidar_mount">
-    <link name="lidar_mount">
-        <visual>
-            <origin rpy="0 0 0" xyz="0 0 0"/>
-            <geometry>
-                <mesh filename="package://jimmbot_description/meshes/ydlidar/ydlidar_mount.stl" scale="0.001 0.001 0.001"/>
-            </geometry>
-        </visual>
-        <collision>
-            <origin rpy="0 0 0" xyz="0 0 0"/>
-            <geometry>
-                <mesh filename="package://jimmbot_description/meshes/ydlidar/ydlidar_mount.stl" scale="0.001 0.001 0.001"/>
-            </geometry>
-        </collision>
-        <xacro:lidar_mount_inertial mass="0.377"/>
-    </link>
-    <joint name="chassis_to_lidar_mount" type="fixed">
-        <origin rpy="0 0 0" xyz="0 0 0.123"/>
-        <parent link="chassis"/>
-        <child link="lidar_mount"/>
-    </joint>
+  <link name="lidar_mount">
+    <visual>
+      <origin rpy="0 0 0" xyz="0 0 0"/>
+      <geometry>
+        <mesh filename="package://jimmbot_description/meshes/ydlidar/ydlidar_mount.stl" scale="0.001 0.001 0.001"/>
+      </geometry>
+    </visual>
+    <collision>
+      <origin rpy="0 0 0" xyz="0 0 0"/>
+      <geometry>
+        <mesh filename="package://jimmbot_description/meshes/ydlidar/ydlidar_mount.stl" scale="0.001 0.001 0.001"/>
+      </geometry>
+    </collision>
+    <xacro:lidar_mount_inertial mass="0.377"/>
+  </link>
+  <joint name="chassis_to_lidar_mount" type="fixed">
+    <origin rpy="0 0 0" xyz="0 0 0.123"/>
+    <parent link="chassis"/>
+    <child link="lidar_mount"/>
+  </joint>
 </xacro:macro>
 <xacro:lidar_mount />
@@ -167,30 +166,42 @@
 <!-- kinect -->
 <xacro:macro name="kinect" params="postfix reflect">
-    <link name="kinect_${postfix}_link">
-        <visual>
-            <origin rpy="0 0 1.5708" xyz="0 0 0"/>
-            <geometry>
-                <mesh filename="package://jimmbot_description/meshes/kinect/kinect.dae" />
-            </geometry>
-        </visual>
-        <collision>
-            <origin rpy="0 0 0" xyz="0 0 0"/>
-            <geometry>
-                <mesh filename="package://jimmbot_description/meshes/kinect/kinect.dae" scale="0.001 0.001 0.001"/>
-            </geometry>
-        </collision>
-        <xacro:differential_inertial mass="0.5"/>
-    </link>
-    <joint name="kinect_${postfix}_optical_joint" type="fixed">
-        <origin xyz="0 0 0" rpy="-1.5708 0 -1.5708"/>
-        <parent link="kinect_${postfix}_link"/>
-        <child link="kinect_${postfix}_optical"/>
+  <link name="kinect_${postfix}_link">
+    <visual>
+      <origin rpy="0 0 1.5708" xyz="0 0 0"/>
+      <geometry>
+        <mesh filename="package://jimmbot_description/meshes/kinect/kinect.dae" />
+      </geometry>
+    </visual>
+    <collision>
+      <origin rpy="0 0 0" xyz="0 0 0"/>
+      <geometry>
+        <mesh filename="package://jimmbot_description/meshes/kinect/kinect.dae" scale="0.001 0.001 0.001"/>
+      </geometry>
+    </collision>
+    <xacro:differential_inertial mass="0.5"/>
+  </link>
+  <joint name="kinect_${postfix}_optical_joint" type="fixed">
+    <origin xyz="0 0 0" rpy="-1.5708 0 -1.5708"/>
+    <parent link="kinect_${postfix}_link"/>
+    <child link="kinect_${postfix}_optical"/>
+  </joint>
+  <link name="kinect_${postfix}_optical"/>
+  <joint name="chassis_to_kinect_${postfix}" type="revolute">
+    <axis xyz="0 ${reflect} 0"/>
+    <limit effort="30.0" lower="-0.523599" upper="0.523599" velocity="0.5"/>
+    <origin rpy="0 0.523599 ${reflect*1.5708-1.5708}" xyz="${reflect*0.25} 0 0.11"/>
+    <parent link="chassis"/>
+    <child link="kinect_${postfix}_link"/>
+  </joint>
+  <transmission name="chassis_to_kinect_${postfix}_trans">
+    <type>transmission_interface/SimpleTransmission</type>
+    <actuator name="chassis_to_kinect_${postfix}_motor">
+      <hardwareInterface>EffortJointInterface</hardwareInterface>
+      <mechanicalReduction>1</mechanicalReduction>
+    </actuator>
+    <joint name="chassis_to_kinect_${postfix}">
+      <hardwareInterface>hardware_interface/PositionJointInterface</hardwareInterface>
     </joint>
-    <link name="kinect_${postfix}_optical"/>
-    <joint name="chassis_to_kinect_${postfix}" type="fixed">
-        <origin rpy="0 0.523599 ${reflect*1.5708-1.5708}" xyz="${reflect*0.25} 0 0.11"/>
-        <parent link="chassis"/>
-        <child link="kinect_${postfix}_link"/>
-    </joint>
+  </transmission>
 </xacro:macro>
 <xacro:kinect postfix="front" reflect="1"/>
@@ -199,36 +210,36 @@
 <!-- boggies -->
 <xacro:macro name="boggie" params="postfix reflect">
-    <link name="boggie_${postfix}_front_rods" />
-    <link name="boggie_${postfix}_back_rods" />
-    <link name="boggie_${postfix}">
-        <visual>
-            <origin rpy="0 0 0" xyz="0 0 0"/>
-            <geometry>
-                <mesh filename="package://jimmbot_description/meshes/boggie/boggie.dae" scale="0.001 0.001 0.001"/>
-            </geometry>
-        </visual>
-        <collision>
-            <origin rpy="0 0 0" xyz="0 0 0"/>
-            <geometry>
-                <mesh filename="package://jimmbot_description/meshes/boggie/boggie.dae" scale="0.001 0.001 0.001"/>
-            </geometry>
-        </collision>
-        <xacro:boggie_inertial mass="6.0"/>
-    </link>
-    <joint name="boggie_${postfix}_front_rods_to_boggie_${postfix}" type="fixed">
-        <origin rpy="0 0 0" xyz="9E-03 -2.5E-03 200E-03"/>
-        <parent link="boggie_${postfix}"/>
-        <child link="boggie_${postfix}_front_rods"/>
-    </joint>
-    <joint name="boggie_${postfix}_back_rods_to_boggie_${postfix}" type="fixed">
-        <origin rpy="0 0 0" xyz="9E-03 -2.5E-03 220E-03"/>
-        <parent link="boggie_${postfix}"/>
-        <child link="boggie_${postfix}_back_rods"/>
-    </joint>
-    <joint name="chassis_to_boggie_${postfix}" type="fixed">
-        <origin rpy="0 0 ${reflect*1.5708}" xyz="${reflect*-1.45758E-03} ${reflect*-201.552E-03} -19.8088E-03"/>
-        <parent link="chassis"/>
-        <child link="boggie_${postfix}"/>
-    </joint>
+  <link name="boggie_${postfix}_front_rods" />
+  <link name="boggie_${postfix}_back_rods" />
+  <link name="boggie_${postfix}">
+    <visual>
+      <origin rpy="0 0 0" xyz="0 0 0"/>
+      <geometry>
+        <mesh filename="package://jimmbot_description/meshes/boggie/boggie.dae" scale="0.001 0.001 0.001"/>
+      </geometry>
+    </visual>
+    <collision>
+      <origin rpy="0 0 0" xyz="0 0 0"/>
+      <geometry>
+        <mesh filename="package://jimmbot_description/meshes/boggie/boggie.dae" scale="0.001 0.001 0.001"/>
+      </geometry>
+    </collision>
+    <xacro:boggie_inertial mass="6.0"/>
+  </link>
+  <joint name="boggie_${postfix}_front_rods_to_boggie_${postfix}" type="fixed">
+    <origin rpy="0 0 0" xyz="9E-03 -2.5E-03 200E-03"/>
+    <parent link="boggie_${postfix}"/>
+    <child link="boggie_${postfix}_front_rods"/>
+  </joint>
+  <joint name="boggie_${postfix}_back_rods_to_boggie_${postfix}" type="fixed">
+    <origin rpy="0 0 0" xyz="9E-03 -2.5E-03 220E-03"/>
+    <parent link="boggie_${postfix}"/>
+    <child link="boggie_${postfix}_back_rods"/>
+  </joint>
+  <joint name="chassis_to_boggie_${postfix}" type="fixed">
+    <origin rpy="0 0 ${reflect*1.5708}" xyz="${reflect*-1.45758E-03} ${reflect*-201.552E-03} -19.8088E-03"/>
+    <parent link="chassis"/>
+    <child link="boggie_${postfix}"/>
+  </joint>
 </xacro:macro>
 <xacro:boggie postfix="right" reflect="1"/>
@@ -237,37 +248,38 @@
 <!-- differential -->
 <xacro:macro name="differential" params="postfix reflect">
-    <link name="differential_left_${postfix}" />
-    <link name="differential_right_${postfix}" />
-    <link name="differential_${postfix}">
-        <visual>
-            <origin rpy="0 0 0" xyz="0 0 0"/>
-            <geometry>
-                <mesh filename="package://jimmbot_description/meshes/differential/differential.stl" scale="0.001 0.001 0.001"/>
-            </geometry>
-        </visual>
-        <collision>
-            <origin rpy="0 0 0" xyz="0 0 0"/>
-            <geometry>
-                <mesh filename="package://jimmbot_description/meshes/differential/differential.stl" scale="0.001 0.001 0.001"/>
-            </geometry>
-        </collision>
-        <xacro:differential_inertial mass="0.8"/>
-    </link>
-    <joint name="differential_${postfix}_to_differential_left_${postfix}" type="fixed">
-        <origin rpy="0 0 0" xyz="120E-03 0 0"/>
-        <parent link="differential_${postfix}"/>
-        <child link="differential_left_${postfix}"/>
-    </joint>
-    <joint name="differential_${postfix}_to_differential_right_${postfix}" type="fixed">
-        <origin rpy="0 0 0" xyz="-120E-03 0 0"/>
-        <parent link="differential_${postfix}"/>
-        <child link="differential_right_${postfix}"/>
-    </joint>
-    <joint name="chassis_to_differential_${postfix}" type="fixed">
-        <limit effort="1000.0" lower="-0.523599" upper="0.523599" velocity="50"/>
-        <origin rpy="0 0 ${reflect*1.5708}" xyz="${reflect*147.5E-03} 0 147.0E-03"/>
-        <parent link="chassis"/>
-        <child link="differential_${postfix}"/>
-    </joint>
+  <link name="differential_left_${postfix}" />
+  <link name="differential_right_${postfix}" />
+  <link name="differential_${postfix}">
+    <visual>
+      <origin rpy="0 0 0" xyz="0 0 0"/>
+      <geometry>
+        <mesh filename="package://jimmbot_description/meshes/differential/differential.stl" scale="0.001 0.001 0.001"/>
+      </geometry>
+    </visual>
+    <collision>
+      <origin rpy="0 0 0" xyz="0 0 0"/>
+      <geometry>
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