Commit message: Initial upgrade of robot to ROS2

File: urdf/jimmbot.gazebo.xacro (robot description, xacro)
@@ -6,4 +6,5 @@
       <always_on>true</always_on>
       <update_rate>20.0</update_rate>
+      <topic>/kinect_front/depth/image_raw</topic>
       <camera>
         <horizontal_fov>${60.0*3.14/180.0}</horizontal_fov>
@@ -18,22 +19,4 @@
         </clip>
       </camera>
-      <plugin name="kinect_front_controller" filename="libgazebo_ros_openni_kinect.so">
-        <cameraName>kinect_front</cameraName>
-        <alwaysOn>true</alwaysOn>
-        <updateRate>10</updateRate>
-        <imageTopicName>rgb/image_color</imageTopicName>
-        <depthImageTopicName>depth/image_raw</depthImageTopicName>
-        <pointCloudTopicName>depth/points</pointCloudTopicName>
-        <cameraInfoTopicName>rgb/camera_info</cameraInfoTopicName>
-        <depthImageCameraInfoTopicName>depth/camera_info</depthImageCameraInfoTopicName>
-        <frameName>kinect_front_optical</frameName>
-        <baseline>0.1</baseline>
-        <distortion_k1>0.0</distortion_k1>
-        <distortion_k2>0.0</distortion_k2>
-        <distortion_k3>0.0</distortion_k3>
-        <distortion_t1>0.0</distortion_t1>
-        <distortion_t2>0.0</distortion_t2>
-        <pointCloudCutoff>0.4</pointCloudCutoff>
-      </plugin>
     </sensor>
   </gazebo>
@@ -43,4 +26,5 @@
       <always_on>true</always_on>
       <update_rate>20.0</update_rate>
+      <topic>/kinect_back/depth/image_raw</topic>
       <camera>
         <horizontal_fov>${60.0*3.14/180.0}</horizontal_fov>
@@ -55,22 +39,4 @@
         </clip>
       </camera>
-      <plugin name="kinect_back_controller" filename="libgazebo_ros_openni_kinect.so">
-        <cameraName>kinect_back</cameraName>
-        <alwaysOn>true</alwaysOn>
-        <updateRate>10</updateRate>
-        <imageTopicName>rgb/image_color</imageTopicName>
-        <depthImageTopicName>depth/image_raw</depthImageTopicName>
-        <pointCloudTopicName>depth/points</pointCloudTopicName>
-        <cameraInfoTopicName>rgb/camera_info</cameraInfoTopicName>
-        <depthImageCameraInfoTopicName>depth/camera_info</depthImageCameraInfoTopicName>
-        <frameName>kinect_back_optical</frameName>
-        <baseline>0.1</baseline>
-        <distortion_k1>0.0</distortion_k1>
-        <distortion_k2>0.0</distortion_k2>
-        <distortion_k3>0.0</distortion_k3>
-        <distortion_t1>0.0</distortion_t1>
-        <distortion_t2>0.0</distortion_t2>
-        <pointCloudCutoff>0.4</pointCloudCutoff>
-      </plugin>
     </sensor>
   </gazebo>
@@ -81,16 +47,5 @@
       <update_rate>50</update_rate>
       <visualize>false</visualize>
-      <topic>__default_topic__</topic>
-      <plugin name="imu_plugin" filename="libgazebo_ros_imu_sensor.so">
-        <topicName>imu</topicName>
-        <bodyName>imu_base</bodyName>
-        <updateRateHZ>50.0</updateRateHZ>
-        <gaussianNoise>0.05</gaussianNoise>
-        <xyzOffset>0 0 0</xyzOffset>
-        <rpyOffset>0 0 0</rpyOffset>
-        <yawOffset>1.5708</yawOffset>
-        <frameName>imu_base</frameName>
-        <initialOrientationAsReference>false</initialOrientationAsReference>
-      </plugin>
+      <topic>/imu</topic>
     </sensor>
   </gazebo>
@@ -99,4 +54,5 @@
       <update_rate>12.0</update_rate>
       <visualize>false</visualize>
+      <topic>/laserscan</topic>
       <ray>
         <scan>
@@ -119,63 +75,27 @@
         </noise>
       </ray>
-      <plugin name="gazebo_ros_ydlidar_controller" filename="libgazebo_ros_laser.so">
-        <topicName>/laserscan</topicName>
-        <frameName>lidar_frame</frameName>
-      </plugin>
     </sensor>
   </gazebo>
-<!-- @todo Check if this or gazebo_imu is better -->
-  <!-- <gazebo>
-    <plugin name="imu_base" filename="libhector_gazebo_ros_imu.so">
-      <serviceName>/imu/calibrate</serviceName>
-      <updateRate>200.0</updateRate>
-      <bodyName>imu_base</bodyName>
-      <frameId>imu_base</frameId>
-      <topicName>imu</topicName>
-      <rpyOffset>0 0 0</rpyOffset>
-      <xyzOffset>0 0 0</xyzOffset>
-      <gaussianNoise>0.00000001</gaussianNoise>
-      <accelDrift>0.00000001 0.00000001 0.00000001</accelDrift>
-      <accelDriftFrequency>0.00000001 0.00000001 0.00000001</accelDriftFrequency>
-      <accelGaussianNoise>0.00000001 0.00000001 0.00000001</accelGaussianNoise>
-      <rateDrift>0.0 0.0 0.0</rateDrift>
-      <rateDriftFrequency>0.0 0.0 0.0</rateDriftFrequency>
-      <rateGaussianNoise>0.0 0.0 0.0</rateGaussianNoise>
-      <headingDrift>0.0 0.0 0.0</headingDrift>
-      <headingDriftFrequency>0.0 0.0 0.0</headingDriftFrequency>
-      <headingGaussianNoise>0.0 0.0 0.0</headingGaussianNoise>
-    </plugin>
-  </gazebo> -->
+  <gazebo reference="gps_front_base">
+    <sensor name="gps_front_sensor" type="navsat">
+      <always_on>true</always_on>
+      <update_rate>50.0</update_rate>
+      <topic>/gps/fix_front</topic>
+    </sensor>
+  </gazebo>
+  <gazebo reference="gps_back_base">
+    <sensor name="gps_back_sensor" type="navsat">
+      <always_on>true</always_on>
+      <update_rate>50.0</update_rate>
+      <topic>/gps/fix_back</topic>
+    </sensor>
+  </gazebo>
   <gazebo>
-    <plugin name="gps_sensor_front" filename="libhector_gazebo_ros_gps.so">
-        <alwayson>true</alwayson>
-        <updaterate>50.0</updaterate>
-        <bodyname>gps_front_base</bodyname>
-        <frameId>gps_front_base</frameId>
-        <topicName>gps/fix_front</topicName>
-        <velocityTopicName>gps/fix_front_velocity</velocityTopicName>
-        <drift>0.001 0.001 0.001</drift>
-        <gaussianNoise>0.05 0.05 0.05</gaussianNoise>
-        <velocityDrift>0.001 0.001 0.001</velocityDrift>
-        <velocityGaussianNoise>0.5 0.5 0.5</velocityGaussianNoise>
+    <plugin filename="libgz_ros2_control-system.so" name="gz_ros2_control::GazeboSimROS2ControlPlugin">
+      <parameters>$(find jimmbot_description)/config/gz_ros2_control.yaml</parameters>
     </plugin>
   </gazebo>
-  <gazebo>
-    <plugin name="gps_sensor_back" filename="libhector_gazebo_ros_gps.so">
-        <alwayson>true</alwayson>
-        <updaterate>50.0</updaterate>
-        <bodyname>gps_back_base</bodyname>
-        <frameId>gps_back_base</frameId>
-        <topicName>/gps/fix_back</topicName>
-        <velocityTopicName>/gps/fix_back_velocity</velocityTopicName>
-        <drift>0.001 0.001 0.001</drift>
-        <gaussianNoise>0.05 0.05 0.05</gaussianNoise>
-        <velocityDrift>0.001 0.001 0.001</velocityDrift>
-        <velocityGaussianNoise>0.5 0.5 0.5</velocityGaussianNoise>
-    </plugin>
-  </gazebo>
-  <gazebo>
-    <plugin name="gazebo_ros_control" filename= "libgazebo_ros_control.so">
-    </plugin>
-  </gazebo>
+  <!-- NOTE: Gazebo Classic ROS plugins were removed for ROS 2 + Gazebo Sim bringup.
+       Equivalent ROS topic delivery is now expected through ros_gz_bridge.
+       Control interfaces now use ros2_control + gz_ros2_control plugin. -->
 </robot>

File: urdf/jimmbot.xacro (robot description, xacro)
@@ -194,14 +194,4 @@
     <child link="kinect_${postfix}_link"/>
   </joint>
-  <transmission name="chassis_to_kinect_${postfix}_trans">
-    <type>transmission_interface/SimpleTransmission</type>
-    <actuator name="chassis_to_kinect_${postfix}_motor">
-      <hardwareInterface>EffortJointInterface</hardwareInterface>
-      <mechanicalReduction>1</mechanicalReduction>
-    </actuator>
-    <joint name="chassis_to_kinect_${postfix}">
-      <hardwareInterface>hardware_interface/PositionJointInterface</hardwareInterface>
-    </joint>
-  </transmission>
 </xacro:macro>
 <xacro:kinect postfix="front" reflect="1"/>
@@ -364,14 +354,4 @@
     <child link="wheel_${side}_${boggie}"/>
   </joint>
-  <transmission name="wheel_axis_${side}_${boggie}_to_wheel_${side}_${boggie}_trans">
-    <type>transmission_interface/SimpleTransmission</type>
-    <actuator name="wheel_axis_${side}_${boggie}_to_wheel_${side}_${boggie}_motor">
-      <hardwareInterface>EffortJointInterface</hardwareInterface>
-      <mechanicalReduction>1</mechanicalReduction>
-    </actuator>
-    <joint name="wheel_axis_${side}_${boggie}_to_wheel_${side}_${boggie}">
-      <hardwareInterface>hardware_interface/VelocityJointInterface</hardwareInterface>
-    </joint>
-  </transmission>
 </xacro:macro>
 <xacro:wheel side="front" boggie="left" across="-1" reflect="1" rotation="1"/>
@@ -380,3 +360,44 @@
 <xacro:wheel side="back" boggie="right" across="-1" reflect="1" rotation="-1"/>
 <!-- end wheels -->
+<ros2_control name="jimmbot_system" type="system">
+  <hardware>
+    <plugin>gz_ros2_control/GazeboSimSystem</plugin>
+  </hardware>
+  <joint name="chassis_to_kinect_front">
+    <command_interface name="position">
+      <param name="min">-0.523599</param>
+      <param name="max">0.523599</param>
+    </command_interface>
+    <state_interface name="position"/>
+    <state_interface name="velocity"/>
+  </joint>
+  <joint name="chassis_to_kinect_back">
+    <command_interface name="position">
+      <param name="min">-0.523599</param>
+      <param name="max">0.523599</param>
+    </command_interface>
+    <state_interface name="position"/>
+    <state_interface name="velocity"/>
+  </joint>
+  <joint name="wheel_axis_front_left_to_wheel_front_left">
+    <command_interface name="velocity"/>
+    <state_interface name="position"/>
+    <state_interface name="velocity"/>
+  </joint>
+  <joint name="wheel_axis_front_right_to_wheel_front_right">
+    <command_interface name="velocity"/>
+    <state_interface name="position"/>
+    <state_interface name="velocity"/>
+  </joint>
+  <joint name="wheel_axis_back_left_to_wheel_back_left">
+    <command_interface name="velocity"/>
+    <state_interface name="position"/>
+    <state_interface name="velocity"/>
+  </joint>
+  <joint name="wheel_axis_back_right_to_wheel_back_right">
+    <command_interface name="velocity"/>
+    <state_interface name="position"/>
+    <state_interface name="velocity"/>
+  </joint>
+</ros2_control>
 </robot>

Commit message: Fixed description model, xacros and launch file

File: urdf/jimmbot.gazebo.xacro (robot description, xacro)
@@ -1,4 +1,5 @@
 <?xml version="1.0"?>
 <robot name="jimmbot_simulation" xmlns:xacro="http://ros.org/wiki/xacro">
+  <xacro:arg name="enable_control" default="true" />
   <!-- Kinect front -->
   <gazebo reference="kinect_front_link">
@@ -91,9 +92,11 @@
     </sensor>
   </gazebo>
-  <gazebo>
-    <plugin filename="libgz_ros2_control-system.so" name="gz_ros2_control::GazeboSimROS2ControlPlugin">
-      <parameters>$(find jimmbot_description)/config/gz_ros2_control.yaml</parameters>
-    </plugin>
-  </gazebo>
+  <xacro:if value="$(arg enable_control)">
+    <gazebo>
+      <plugin filename="libgz_ros2_control-system.so" name="gz_ros2_control::GazeboSimROS2ControlPlugin">
+        <parameters>$(find jimmbot_controller)/config/gz_ros2_control.yaml</parameters>
+      </plugin>
+    </gazebo>
+  </xacro:if>
   <!-- NOTE: Gazebo Classic ROS plugins were removed for ROS 2 + Gazebo Sim bringup.
        Equivalent ROS topic delivery is now expected through ros_gz_bridge.

File: urdf/jimmbot.xacro (robot description, xacro)
@@ -1,6 +1,25 @@
 <?xml version="1.0" ?>
 <robot name="jimmbot" xmlns:xacro="http://www.ros.org/wiki/xacro">
+<xacro:arg name="enable_control" default="true" />
 <xacro:include filename="$(find jimmbot_description)/urdf/jimmbot_inertias.xacro" />
 <xacro:include filename="$(find jimmbot_description)/urdf/jimmbot.gazebo.xacro" />
+<material name="jimmbot_chassis_gray">
+  <color rgba="0.20 0.23 0.26 1.0"/>
+</material>
+<material name="jimmbot_sensor_black">
+  <color rgba="0.08 0.09 0.10 1.0"/>
+</material>
+<material name="jimmbot_metal">
+  <color rgba="0.58 0.61 0.66 1.0"/>
+</material>
+<material name="jimmbot_trim_orange">
+  <color rgba="0.86 0.42 0.18 1.0"/>
+</material>
+<material name="jimmbot_rubber">
+  <color rgba="0.11 0.11 0.12 1.0"/>
+</material>
+<material name="jimmbot_sensor_light">
+  <color rgba="0.74 0.76 0.79 1.0"/>
+</material>
 <!-- dummy base_link -->
 <link name="base_link" />
@@ -17,4 +36,5 @@
       <mesh filename="package://jimmbot_description/meshes/chassis/chassis.stl" scale="0.001 0.001 0.001"/>
     </geometry>
+    <material name="jimmbot_chassis_gray"/>
   </visual>
   <collision>
@@ -36,4 +56,5 @@
         <box size="0.037 0.052 0.035" />
       </geometry>
+      <material name="jimmbot_sensor_black"/>
     </visual>
     <!-- IMU is inside chassis, no need for collision, chassis collision will handle all inside the chassis -->
@@ -147,4 +168,5 @@
         <mesh filename="package://jimmbot_description/meshes/ydlidar/ydlidar_mount.stl" scale="0.001 0.001 0.001"/>
       </geometry>
+      <material name="jimmbot_metal"/>
     </visual>
     <collision>
@@ -170,5 +192,5 @@
       <origin rpy="0 0 1.5708" xyz="0 0 0"/>
       <geometry>
-        <mesh filename="package://jimmbot_description/meshes/kinect/kinect.dae" />
+        <mesh filename="package://jimmbot_description/meshes/kinect/kinect.dae" scale="0.001 0.001 0.001" />
       </geometry>
     </visual>
@@ -246,4 +268,5 @@
         <mesh filename="package://jimmbot_description/meshes/differential/differential.stl" scale="0.001 0.001 0.001"/>
       </geometry>
+      <material name="jimmbot_metal"/>
     </visual>
     <collision>
@@ -286,4 +309,5 @@
         <mesh filename="package://jimmbot_description/meshes/differential/differential_rod.stl" scale="0.01 0.01 0.01"/>
       </geometry>
+      <material name="jimmbot_metal"/>
     </visual>
     <collision>

Commit message: Fixed launchfile and kinect model,

File: urdf/jimmbot.gazebo.xacro (robot description, xacro)
@@ -1,11 +1,9 @@
 <?xml version="1.0"?>
 <robot name="jimmbot_simulation" xmlns:xacro="http://ros.org/wiki/xacro">
-  <xacro:arg name="enable_control" default="true" />
-  <!-- Kinect front -->
+  <!-- Kinect front (Gazebo Sim format) -->
   <gazebo reference="kinect_front_link">
-    <sensor type="depth" name="kinect_front">
+    <sensor name="kinect_front" type="camera">
       <always_on>true</always_on>
       <update_rate>20.0</update_rate>
-      <topic>/kinect_front/depth/image_raw</topic>
       <camera>
         <horizontal_fov>${60.0*3.14/180.0}</horizontal_fov>
@@ -22,10 +20,9 @@
     </sensor>
   </gazebo>
-  <!-- Kinect back -->
+  <!-- Kinect back (Gazebo Sim format) -->
   <gazebo reference="kinect_back_link">
-    <sensor type="depth" name="kinect_back">
+    <sensor name="kinect_back" type="camera">
       <always_on>true</always_on>
       <update_rate>20.0</update_rate>
-      <topic>/kinect_back/depth/image_raw</topic>
       <camera>
         <horizontal_fov>${60.0*3.14/180.0}</horizontal_fov>
@@ -48,13 +45,12 @@
       <update_rate>50</update_rate>
       <visualize>false</visualize>
-      <topic>/imu</topic>
     </sensor>
   </gazebo>
   <gazebo reference="lidar_frame">
-    <sensor type="ray" name="ydlidar_sensor">
+    <sensor type="lidar" name="ydlidar_sensor">
+      <always_on>true</always_on>
       <update_rate>12.0</update_rate>
       <visualize>false</visualize>
-      <topic>/laserscan</topic>
-      <ray>
+      <lidar>
         <scan>
           <horizontal>
@@ -75,5 +71,5 @@
           <stddev>0.01</stddev>
         </noise>
-      </ray>
+      </lidar>
     </sensor>
   </gazebo>
@@ -82,5 +78,4 @@
       <always_on>true</always_on>
       <update_rate>50.0</update_rate>
-      <topic>/gps/fix_front</topic>
     </sensor>
   </gazebo>
@@ -89,5 +84,4 @@
       <always_on>true</always_on>
       <update_rate>50.0</update_rate>
-      <topic>/gps/fix_back</topic>
     </sensor>
   </gazebo>
@@ -95,13 +89,7 @@
     <plugin filename="ignition-gazebo-joint-state-publisher-system" name="ignition::gazebo::systems::JointStatePublisher"/>
   </gazebo>
-  <xacro:if value="$(arg enable_control)">
-    <gazebo>
-      <plugin filename="libgz_ros2_control-system.so" name="gz_ros2_control::GazeboSimROS2ControlPlugin">
-        <parameters>$(find jimmbot_controller)/config/gz_ros2_control.yaml</parameters>
-      </plugin>
-    </gazebo>
-  </xacro:if>
-  <!-- NOTE: Gazebo Classic ROS plugins were removed for ROS 2 + Gazebo Sim bringup.
-       Equivalent ROS topic delivery is now expected through ros_gz_bridge.
-       Control interfaces now use ros2_control + gz_ros2_control plugin. -->
+  <!-- NOTE: Control plugin is configured by jimmbot_gazebo launch files.
+       Gazebo Classic ROS plugins were removed for ROS 2 + Gazebo Sim bringup.
+       Equivalent ROS topic delivery is now handled through ros_gz_bridge.
+       Control interfaces use ros2_control + gz_ros2_control plugin configured in gazebo launches. -->
 </robot>

File: urdf/jimmbot.xacro (robot description, xacro)
@@ -1,7 +1,6 @@
 <?xml version="1.0" ?>
 <robot name="jimmbot" xmlns:xacro="http://www.ros.org/wiki/xacro">
-<xacro:arg name="enable_control" default="true" />
-<xacro:include filename="$(find jimmbot_description)/urdf/jimmbot_inertias.xacro" />
-<xacro:include filename="$(find jimmbot_description)/urdf/jimmbot.gazebo.xacro" />
+<xacro:include filename="jimmbot_inertias.xacro" />
+<xacro:include filename="jimmbot.gazebo.xacro" />
 <material name="jimmbot_chassis_gray">
   <color rgba="0.20 0.23 0.26 1.0"/>
@@ -192,11 +191,11 @@
       <origin rpy="0 0 1.5708" xyz="0 0 0"/>
       <geometry>
-        <mesh filename="package://jimmbot_description/meshes/kinect/kinect.dae" scale="0.001 0.001 0.001" />
-      </geometry>
-    </visual>
-    <collision>
-      <origin rpy="0 0 0" xyz="0 0 0"/>
-      <geometry>
-        <mesh filename="package://jimmbot_description/meshes/kinect/kinect.dae" scale="0.001 0.001 0.001"/>
+        <mesh filename="package://jimmbot_description/meshes/kinect/kinect.dae" />
+      </geometry>
+    </visual>
+    <collision>
+      <origin rpy="0 0 0" xyz="0 0 0"/>
+      <geometry>
+        <mesh filename="package://jimmbot_description/meshes/kinect/kinect.dae"/>
       </geometry>
     </collision>
